Commit message: Implement odometry

File: src/exr1_description/urdf/exr1.urdf.xacro (robot description, xacro)
@@ -6,5 +6,5 @@
   <xacro:include filename="$(find exr1_description)/urdf/utils.xacro" />
   <xacro:include filename="$(find exr1_description)/urdf/wheel.urdf.xacro" />
-  <link name="base_link" />
+  <link name="base_footprint" />
   <joint name="body_joint" type="fixed">
     <parent link="base_link" />
@@ -27,10 +27,10 @@
     </visual>
   </link>
-  <joint name="base_footprint_joint" type="fixed">
-    <parent link="base_link" />
-    <child link="base_footprint" />
+  <joint name="base_link_joint" type="fixed">
+    <parent link="base_footprint" />
+    <child link="base_link" />
     <origin xyz="0 0 0" rpy="0 0 0" />
   </joint>
-  <link name="base_footprint" />
+  <link name="base_link" />
   <xacro:wheel name="front_left">
     <origin xyz="${wheel_separation} ${wheel_separation} ${wheel_radius}"
@@ -60,5 +60,5 @@
       <linear_damping>50</linear_damping>
       <angular_damping>5</angular_damping>
-      <base_link>base_link</base_link>
+      <base_link>base_footprint</base_link>
       <!-- <mass>30</mass> -->
       <!-- <center_of_mass>${-wheel_separation/2.0*(1.0-cos(pi/3))} 0</center_of_mass> -->

Commit message: Adjust URDF

File: src/exr1_description/urdf/exr1.urdf.xacro (robot description, xacro)
@@ -1,10 +1,16 @@
 <?xml version="1.0"?>
 <robot name="exr1" xmlns:xacro="http://ros.org/wiki/xacro">
-  <xacro:property name="wheel_separation" value="0.6" />
-  <xacro:property name="wheel_radius" value="0.1" />
-  <xacro:property name="body_height" value="0.01" />
+  <xacro:property name="wheel_separation" value="0.35" />
+  <xacro:property name="wheel_radius" value="0.05" />
+  <xacro:property name="body_height" value="0.025" />
   <xacro:include filename="$(find exr1_description)/urdf/utils.xacro" />
   <xacro:include filename="$(find exr1_description)/urdf/wheel.urdf.xacro" />
   <link name="base_footprint" />
+  <joint name="base_link_joint" type="fixed">
+    <parent link="base_footprint" />
+    <child link="base_link" />
+    <origin xyz="0 0 0" rpy="0 0 0" />
+  </joint>
+  <link name="base_link" />
   <joint name="body_joint" type="fixed">
     <parent link="base_link" />
@@ -27,23 +33,17 @@
     </visual>
   </link>
-  <joint name="base_link_joint" type="fixed">
-    <parent link="base_footprint" />
-    <child link="base_link" />
-    <origin xyz="0 0 0" rpy="0 0 0" />
-  </joint>
-  <link name="base_link" />
-  <xacro:wheel name="front_left">
+  <xacro:wheel name="front_left" radius="${wheel_radius}">
     <origin xyz="${wheel_separation} ${wheel_separation} ${wheel_radius}"
       rpy="${-pi/2} 0 ${1*pi/4+pi/2}" />
   </xacro:wheel>
-  <xacro:wheel name="rear_left">
+  <xacro:wheel name="rear_left" radius="${wheel_radius}">
     <origin xyz="${-wheel_separation} ${wheel_separation} ${wheel_radius}"
       rpy="${-pi/2} 0 ${3*pi/4+pi/2}" />
   </xacro:wheel>
-  <xacro:wheel name="rear_right">
+  <xacro:wheel name="rear_right" radius="${wheel_radius}">
     <origin xyz="${-wheel_separation} ${-wheel_separation} ${wheel_radius}"
       rpy="${-pi/2} 0 ${5*pi/4+pi/2}" />
   </xacro:wheel>
-  <xacro:wheel name="front_right">
+  <xacro:wheel name="front_right" radius="${wheel_radius}">
     <origin xyz="${wheel_separation} ${-wheel_separation} ${wheel_radius}"
       rpy="${-pi/2} 0 ${7*pi/4+pi/2}" />
@@ -51,8 +51,4 @@
   <gazebo>
     <plugin filename="libexr1_sim_plugin.so" name="exr1_gz::Exr1System">
-      <!-- <wheel0_joint>front_left_wheel_joint</wheel0_joint> -->
-      <!-- <wheel1_joint>rear_left_wheel_joint</wheel1_joint> -->
-      <!-- <wheel2_joint>rear_right_wheel_joint</wheel2_joint> -->
-      <!-- <wheel3_joint>front_right_wheel_joint</wheel3_joint> -->
       <max_wheel_torque>10.0</max_wheel_torque>
       <wheel_radius>${wheel_radius}</wheel_radius>
@@ -61,14 +57,4 @@
       <angular_damping>5</angular_damping>
       <base_link>base_footprint</base_link>
-      <!-- <mass>30</mass> -->
-      <!-- <center_of_mass>${-wheel_separation/2.0*(1.0-cos(pi/3))} 0</center_of_mass> -->
-      <!-- <center_of_mass>0 0</center_of_mass> -->
-      <!-- <moment_of_inertia>2.29</moment_of_inertia> -->
-      <!-- <linear_kp>1</linear_kp> -->
-      <!-- <linear_ki>0</linear_ki> -->
-      <!-- <linear_kd>0</linear_kd> -->
-      <!-- <angular_kp>0</angular_kp> -->
-      <!-- <angular_ki>0</angular_ki> -->
-      <!-- <angular_kd>0</angular_kd> -->
     </plugin>
   </gazebo>

File: src/exr1_description/urdf/utils.xacro (robot description, xacro)
@@ -1,34 +1,36 @@
 <?xml version="1.0"?>
-<robot xmlns:xacro="http://www.ros.org/wiki/xacro" >
-    <!-- From https://github.com/joshnewans/urdf_example/blob/main/description/example_include.xacro -->
-    <!-- This file is not a robot in and of itself, it just contains some useful tags that could be included in any robot -->
-    <!-- Specify some standard inertial calculations https://en.wikipedia.org/wiki/List_of_moments_of_inertia -->
-    <!-- These make use of xacro's mathematical functionality -->
-    <xacro:macro name="inertial_sphere" params="mass radius *origin">
-        <inertial>
-            <xacro:insert_block name="origin"/>
-            <mass value="${mass}" />
-            <inertia ixx="${(2/5) * mass * (radius*radius)}" ixy="0.0" ixz="0.0"
-                    iyy="${(2/5) * mass * (radius*radius)}" iyz="0.0"
-                    izz="${(2/5) * mass * (radius*radius)}" />
-        </inertial>
-    </xacro:macro>
-    <xacro:macro name="inertial_box" params="mass x y z *origin">
-        <inertial>
-            <xacro:insert_block name="origin"/>
-            <mass value="${mass}" />
-            <inertia ixx="${(1/12) * mass * (y*y+z*z)}" ixy="0.0" ixz="0.0"
-                    iyy="${(1/12) * mass * (x*x+z*z)}" iyz="0.0"
-                    izz="${(1/12) * mass * (x*x+y*y)}" />
-        </inertial>
-    </xacro:macro>
-    <xacro:macro name="inertial_cylinder" params="mass length radius">
-        <inertial>
-            <xacro:insert_block name="origin"/>
-            <mass value="${mass}" />
-            <inertia ixx="${(1/12) * mass * (3*radius*radius + length*length)}" ixy="0.0" ixz="0.0"
-                    iyy="${(1/12) * mass * (3*radius*radius + length*length)}" iyz="0.0"
-                    izz="${(1/2) * mass * (radius*radius)}" />
-        </inertial>
-    </xacro:macro>
+<robot xmlns:xacro="http://www.ros.org/wiki/xacro">
+  <!-- From https://github.com/joshnewans/urdf_example/blob/main/description/example_include.xacro -->
+  <!-- This file is not a robot in and of itself, it just contains some useful tags that could be
+  included in any robot -->
+  <!-- Specify some standard inertial calculations
+  https://en.wikipedia.org/wiki/List_of_moments_of_inertia -->
+  <!-- These make use of xacro's mathematical functionality -->
+  <xacro:macro name="inertial_sphere" params="mass radius *origin">
+    <inertial>
+      <xacro:insert_block name="origin" />
+      <mass value="${mass}" />
+      <inertia ixx="${(2/5) * mass * (radius*radius)}" ixy="0.0" ixz="0.0"
+        iyy="${(2/5) * mass * (radius*radius)}" iyz="0.0"
+        izz="${(2/5) * mass * (radius*radius)}" />
+    </inertial>
+  </xacro:macro>
+  <xacro:macro name="inertial_box" params="mass x y z *origin">
+    <inertial>
+      <xacro:insert_block name="origin" />
+      <mass value="${mass}" />
+      <inertia ixx="${(1/12) * mass * (y*y+z*z)}" ixy="0.0" ixz="0.0"
+        iyy="${(1/12) * mass * (x*x+z*z)}" iyz="0.0"
+        izz="${(1/12) * mass * (x*x+y*y)}" />
+    </inertial>
+  </xacro:macro>
+  <xacro:macro name="inertial_cylinder" params="mass length radius">
+    <inertial>
+      <xacro:insert_block name="origin" />
+      <mass value="${mass}" />
+      <inertia ixx="${(1/12) * mass * (3*radius*radius + length*length)}" ixy="0.0" ixz="0.0"
+        iyy="${(1/12) * mass * (3*radius*radius + length*length)}" iyz="0.0"
+        izz="${(1/2) * mass * (radius*radius)}" />
+    </inertial>
+  </xacro:macro>
 </robot>

File: src/exr1_description/urdf/wheel.urdf.xacro (robot description, xacro)
@@ -1,7 +1,6 @@
 <?xml version="1.0"?>
 <robot xmlns:xacro="http://ros.org/wiki/xacro" xmlns:gz="http://gazebosim.org/schema">
-  <xacro:macro name="wheel" params="name parent_link:=base_link *origin">
+  <xacro:macro name="wheel" params="name radius parent_link:=base_link *origin">
     <xacro:property name="mass" value="0.5" />
-    <xacro:property name="radius" value="0.2" />
     <xacro:property name="width" value="0.06" />
     <xacro:property name="wheel_link_name" value="${name}_wheel" />
@@ -11,5 +10,4 @@
       <child link="${wheel_link_name}" />
       <xacro:insert_block name="origin" />
-      <!-- <axis xyz="0 0 1" /> -->
     </joint>
     <link name="${wheel_link_name}">

Commit message: Add lidar

File: src/exr1_description/urdf/exr1.urdf.xacro (robot description, xacro)
@@ -6,4 +6,5 @@
   <xacro:include filename="$(find exr1_description)/urdf/utils.xacro" />
   <xacro:include filename="$(find exr1_description)/urdf/wheel.urdf.xacro" />
+  <xacro:include filename="$(find exr1_description)/urdf/ld06_lidar.urdf.xacro" />
   <link name="base_footprint" />
   <joint name="base_link_joint" type="fixed">
@@ -49,4 +50,10 @@
       rpy="${-pi/2} 0 ${7*pi/4+pi/2}" />
   </xacro:wheel>
+  <xacro:ld06_lidar name="left_lidar" topic="scan_left">
+    <origin xyz="0 0.4 0.1" rpy="0 0 0" />
+  </xacro:ld06_lidar>
+  <xacro:ld06_lidar name="right_lidar" topic="scan_right">
+    <origin xyz="0 -0.4 0.1" rpy="0 0 ${pi}" />
+  </xacro:ld06_lidar>
   <gazebo>
     <plugin filename="libexr1_sim_plugin.so" name="exr1_gz::Exr1System">
