Commit message: Add ransac_localization

File: src/exr1_bringup/urdf/field.urdf.xacro (robot description, xacro)
@@ -2,5 +2,5 @@
 <robot name="field" xmlns:xacro="http://ros.org/wiki/xacro">
   <xacro:property name="field_width" value="8.0" />
-  <xacro:property name="field_height" value="3.0" />
+  <xacro:property name="field_height" value="8.0" />
   <xacro:property name="fence_height" value="0.15" />
   <xacro:property name="fence_width" value="0.15" />

File: src/exr1_description/urdf/ld06_lidar.urdf.xacro (robot description, xacro)
@@ -58,5 +58,5 @@
             <type>gaussian</type>
             <mean>0.0</mean>
-            <stddev>0.03</stddev>
+            <stddev>0.01</stddev>
           </noise>
         </lidar>
